File: Halloween-Controller/Halloween-Controller.sch (KiCad schematic (older format))
At the start: 30 parts, among them IC1 ATmega328_B, J1 Neopixel_A, J2 Conn_FTDI, J3 Conn_Sensors, J4 Neopixel_B, J5 Neopixel_C, J6 Conn_Exp, J7 Neopixel_D, J8 Conn_GPIO_IN, SW1 SW_SPST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

Commit message: WIP....
Parts:
- C1, C2, C3, C4: symbol CE_Capacitor:C -> Halloween-Controller-rescue:C-CE_Capacitor
- IC1: symbol MFS_Microcontrollers:ATmega328_B -> Halloween-Controller-rescue:ATmega328_B-MFS_Microcontrollers
- R1, R2, R3, R4, R5, R6, R7, R8: symbol CE_Resistor:R -> Halloween-Controller-rescue:R-CE_Resistor
- VTR1: symbol MFS_Power:Adafruit_PowerBoost_1000C -> Halloween-Controller-rescue:Adafruit_PowerBoost_1000C-MFS_Power
- Y1: symbol CE_Crystal:Crystal -> Halloween-Controller-rescue:Crystal-CE_Crystal
Changed lines of the file:
@@
 $EndDescr
 $Comp
-L MFS_Microcontrollers:ATmega328_B IC1
+L Halloween-Controller-rescue:ATmega328_B-MFS_Microcontrollers IC1
 U 1 1 5C5F55C5
 P 5800 2300
@@
 $EndComp
 $Comp
-L CE_Crystal:Crystal Y1
+L Halloween-Controller-rescue:Crystal-CE_Crystal Y1
 U 1 1 5C5F566A
 P 4200 2300
@@
 $EndComp
 $Comp
-L CE_Capacitor:C C2
+L Halloween-Controller-rescue:C-CE_Capacitor C2
 U 1 1 5C5F56EA
 P 3850 2100
@@
 $EndComp
 $Comp
-L CE_Capacitor:C C3
+L Halloween-Controller-rescue:C-CE_Capacitor C3
 U 1 1 5C5F57A4
 P 3850 2500
@@
 $EndComp
 $Comp
-L CE_VirtualSymbols:GND #PWR014
+L Halloween-Controller-rescue:GND-CE_VirtualSymbols #PWR014
 U 1 1 5C5F57F9
 P 3600 2600
@@
 $EndComp
 $Comp
-L CE_VirtualSymbols:GND #PWR09
+L Halloween-Controller-rescue:GND-CE_VirtualSymbols #PWR09
 U 1 1 5C5F5B3D
 P 4200 1700
@@
 	5000 1250 5000 1850
 $Comp
-L CE_Capacitor:C C1
+L Halloween-Controller-rescue:C-CE_Capacitor C1
 U 1 1 5C5F6D87
 P 4200 1100
@@
 	5100 1750 5300 1750
 $Comp
-L CE_Resistor:R R3
+L Halloween-Controller-rescue:R-CE_Resistor R3
 U 1 1 5C5FB22E
 P 5400 1100
@@
 	3600 2500 3600 2600
 $Comp
-L CE_VirtualSymbols:GND #PWR017
+L Halloween-Controller-rescue:GND-CE_VirtualSymbols #PWR017
 U 1 1 5C5FF293
 P 5800 3250
@@
 $EndComp
 $Comp
-L CE_VirtualSymbols:GND #PWR022
+L Halloween-Controller-rescue:GND-CE_VirtualSymbols #PWR022
 U 1 1 5C60110C
 P 3550 7200
@@
 $EndComp
 $Comp
-L CE_Capacitor:C C4
+L Halloween-Controller-rescue:C-CE_Capacitor C4
 U 1 1 5C601140
 P 3550 7000
@@
 	5200 2550 5300 2550
 $Comp
-L CE_Resistor:R R2
+L Halloween-Controller-rescue:R-CE_Resistor R2
 U 1 1 5C61AA52
 P 7950 1100
@@
 $EndComp
 $Comp
-L CE_VirtualSymbols:GND #PWR04
+L Halloween-Controller-rescue:GND-CE_VirtualSymbols #PWR04
 U 1 1 5C61C3A3
 P 8250 1300
@@
 GPIO_2
 $Comp
-L CE_Resistor:R R5
+L Halloween-Controller-rescue:R-CE_Resistor R5
 U 1 1 5C629098
 P 7950 2100
@@
 $EndComp
 $Comp
-L CE_VirtualSymbols:GND #PWR011
+L Halloween-Controller-rescue:GND-CE_VirtualSymbols #PWR011
 U 1 1 5C62909E
 P 8250 2300
@@
 GPIO_3
 $Comp
-L CE_Resistor:R R7
+L Halloween-Controller-rescue:R-CE_Resistor R7
 U 1 1 5C62CDA2
 P 7950 3100
@@
 $EndComp
 $Comp
-L CE_VirtualSymbols:GND #PWR016
+L Halloween-Controller-rescue:GND-CE_VirtualSymbols #PWR016
 U 1 1 5C62CDA8
 P 8250 3300
@@
 GPIO_4
 $Comp
-L CE_Resistor:R R8
+L Halloween-Controller-rescue:R-CE_Resistor R8
 U 1 1 5C62CDC0
 P 7950 4100
@@
 $EndComp
 $Comp
-L CE_VirtualSymbols:GND #PWR023
+L Halloween-Controller-rescue:GND-CE_VirtualSymbols #PWR023
 U 1 1 5C62CDC6
 P 8250 4300
@@
 GPIO_10
 $Comp
-L CE_Resistor:R R1
+L Halloween-Controller-rescue:R-CE_Resistor R1
 U 1 1 5C6775C2
 P 2200 1200
@@
 $EndComp
 $Comp
-L CE_VirtualSymbols:GND #PWR03
+L Halloween-Controller-rescue:GND-CE_VirtualSymbols #PWR03
 U 1 1 5C6775C8
 P 1900 1400
@@
 AIO_0
 $Comp
-L CE_VirtualSymbols:GND #PWR010
+L Halloween-Controller-rescue:GND-CE_VirtualSymbols #PWR010
 U 1 1 5C6775E6
 P 1900 2400
@@
 AIO_1
 $Comp
-L CE_VirtualSymbols:GND #PWR015
+L Halloween-Controller-rescue:GND-CE_VirtualSymbols #PWR015
 U 1 1 5C677604
 P 1900 3400
@@
 AIO_2
 $Comp
-L CE_VirtualSymbols:GND #PWR021
+L Halloween-Controller-rescue:GND-CE_VirtualSymbols #PWR021
 U 1 1 5C677622
 P 2350 4800
@@
 AIO_3
 $Comp
-L CE_Resistor:R R4
+L Halloween-Controller-rescue:R-CE_Resistor R4
 U 1 1 5C67F86D
 P 2200 2200
@@
 $EndComp
 $Comp
-L CE_Resistor:R R6
+L Halloween-Controller-rescue:R-CE_Resistor R6
 U 1 1 5C67F915
 P 2200 3200
@@
 (future use)
 $Comp
-L CE_VirtualSymbols:GND #PWR025
+L Halloween-Controller-rescue:GND-CE_VirtualSymbols #PWR025
 U 1 1 5C6962F0
 P 3000 6900
@@
 	1650 3100 1900 3100
 $Comp
-L CE_VirtualSymbols:GND #PWR0101
+L Halloween-Controller-rescue:GND-CE_VirtualSymbols #PWR0101
 U 1 1 5C6D08D8
 P 5800 7550
@@
 	5800 7450 5800 7550
 $Comp
-L MFS_Power:Adafruit_PowerBoost_1000C VTR1
+L Halloween-Controller-rescue:Adafruit_PowerBoost_1000C-MFS_Power VTR1
 U 1 1 5C5FB45B
 P 2200 7150
@@
 $EndComp
 $Comp
-L CE_VirtualSymbols:GND #PWR026
+L Halloween-Controller-rescue:GND-CE_VirtualSymbols #PWR026
 U 1 1 5C61A1F3
 P 850 7150
