File: Halloween-Soundboard/Halloween-Soundboard.sch (KiCad schematic (older format))
At the start: 6 parts, among them U1 MCP23008-E_P

Commit message: WIP....
Parts:
- ADA1: symbol MFS_Microcontrollers:Adafruit_AudioFX -> Halloween-Soundboard-rescue:Adafruit_AudioFX-MFS_Microcontrollers
- U1: symbol MFS_Transistors:MCP23008-E_P -> Halloween-Soundboard-rescue:MCP23008-E_P-MFS_Transistors
Changed lines of the file:
@@
 $EndComp
 $Comp
-L CE_VirtualSymbols:GND #PWR0101
+L Halloween-Soundboard-rescue:GND-CE_VirtualSymbols #PWR0101
 U 1 1 5C6D08D8
 P 5800 7550
@@
 	5800 7450 5800 7550
 $Comp
-L MFS_Microcontrollers:Adafruit_AudioFX ADA1
+L Halloween-Soundboard-rescue:Adafruit_AudioFX-MFS_Microcontrollers ADA1
 U 1 1 5C605CF2
 P 5050 3250
@@
 $EndComp
 $Comp
-L MFS_Transistors:MCP23008-E_P U1
+L Halloween-Soundboard-rescue:MCP23008-E_P-MFS_Transistors U1
 U 1 1 5C605F7E
 P 3750 3000
